Commit message: feat(scout): 整合 Scout 控制和模拟功能
- 更新 Scout 控制配置，增加新的控制器和参数
- 重构 Scout 描述包，添加依赖和优化构建过程
- 修改 URDF 文件，调整惯性参数和关节起源
- 更新 Gazebo 启动脚本，使用新的控制器和参数

File: scout_description/urdf/scout_mini_backup.urdf (robot description, URDF)
Before this commit: robot scout_mini, 7 links, 6 joints
Links:
- added link inertial_link, mass 30
- link base_link: mass 30 -> None
- link laser_link: geometry collision cylinder length=0.1 radius=0.06; visual cylinder length=0.01 radius=0.01
Joints:
- added joint inertial_joint: type fixed, parent base_link, child inertial_link, origin xyz=0 0 0 rpy=0 0 0
