Commit message: test(scout): add diff drive controller and update launch files
- Add diff drive controller configuration for Scout robot
- Update launch files to use new controller
- Rename controller configuration file
- Adjust joint names in URDF to match new controller
- Remove unused backup URDF file

File: scout_description/urdf/scout_mini.urdf (robot description, URDF)
Before this commit: robot scout_mini, 8 links, 7 joints
Joints:
- removed joint front_left_wheel
- removed joint front_right_wheel
- removed joint rear_left_wheel
- removed joint rear_right_wheel
- added joint front_left_wheel_joint: type continuous, parent base_link, child front_left_wheel_link, origin xyz=0.2319755 0.2082515 -0.100998 rpy=-1.57 0 0, axis 0 0 -1
- added joint front_right_wheel_joint: type continuous, parent base_link, child front_right_wheel_link, origin xyz=0.2319755 -0.2082515 -0.099998 rpy=1.57 0 0, axis 0 0 -1
- added joint rear_left_wheel_joint: type continuous, parent base_link, child rear_left_wheel_link, origin xyz=-0.2319755 0.2082515 -0.100998 rpy=-1.57 0 0, axis 0 0 -1
- added joint rear_right_wheel_joint: type continuous, parent base_link, child rear_right_wheel_link, origin xyz=-0.2319755 -0.2082515 -0.099998 rpy=1.57 0 0, axis 0 0 -1

Commit message: Add URDF and Xacro files for fishros_robot and lidar_robot configurations
- Created fishros_robot.urdf.xacro to define the robot structure, including sensors (camera, laser, IMU) and actuators (wheels, casters).
- Added lidar_robot.urdf.xacro for a simple robot model with a lidar sensor.
- Implemented gazebo_control_plugin.xacro for integrating ROS2 control with Gazebo simulation.
- Developed gazebo_sensor_plugin.xacro to manage sensor configurations for laser and IMU.
- Introduced ign_sensor_plugin.xacro for additional sensor functionalities.
- Created lidar_sensor.xacro for lidar sensor specifications.
- Added camera.urdf.xacro for camera module integration.
- Developed imu.urdf.xacro for IMU sensor specifications.
- Created laser.urdf.xacro for laser sensor integration.
- Added lidar.xacro for lidar sensor configuration with Gazebo.
- Implemented rgbd_camera.xacro for RGBD camera specifications.
- Generated text.urdf as an autogenerated file from the Xacro definitions.

File: scout_description/urdf/scout_mini.urdf (robot description, URDF)
Before this commit: robot scout_mini, 7 links, 6 joints
Links:
- removed link camera_link
- removed link laser_link
Joints:
- removed joint camera_joint
- removed joint laser_joint

File: scout_description/urdf/scout_mini.urdf.xacro (robot description, xacro)
@@ -1,117 +1,108 @@
 <?xml version="1.0"?>
-<robot name="scout_mini"
-    xmlns:xacro="http://ros.org/wiki/xacro">
-    <xacro:arg name="robot_namespace" default="/" />
-    <xacro:arg name="urdf_extras" default="empty.urdf" />
-    <xacro:include filename="$(find scout_description)/urdf/scout_mini_wheel_1.xacro" />
-    <xacro:include filename="$(find scout_description)/urdf/scout_mini_wheel_2.xacro" />
-    <xacro:include filename="$(find scout_description)/urdf/scout_mini_wheel_3.xacro" />
-    <xacro:include filename="$(find scout_description)/urdf/scout_mini_wheel_4.xacro" />
-    <!-- Variables -->
-    <xacro:property name="M_PI" value="3.14159"/>
-    <!-- Vehicle Geometries -->
-    <xacro:property name="base_x_size" value="0.6200000" />
-    <xacro:property name="base_y_size" value="0.585000" />
-    <xacro:property name="base_z_size" value="0.235000" />
-    <xacro:property name="wheelbase" value="0.3132556"/>
-   <xacro:property name="track" value="0.4563536" />
-   <xacro:property name="wheel_vertical_offset" value="-0.077" />
-    <xacro:property name="wheel_diameter" value="0.16" />
-    <xacro:property name="wheel_width" value="0.084" />
-<!--    <xacro:property name="track" value="0.3426" />
-    <xacro:property name="wheelbase" value="0.3181"/>
-    <xacro:property name="wheel_vertical_offset" value="-0.160000047342231" />-->
-    <xacro:property name="wheel_length" value="0.8e-01" />
-    <xacro:property name="wheel_radius" value="1.600e-01" />
-    <!-- Base link -->
-    <link name="base_link">
-        <visual>
-            <!--origin xyz="-0.0145261552504705 0.0231316650320557 0.00586280190939592" rpy="0 0 0" /-->
-            <origin xyz="0.015 0.0231316650320557 0" rpy="0 0 0"/>
-            <!--<origin
-              xyz="-0.0145261552504705 0.0231316650320557 0.00586280190939592"
-              rpy="0 0 0" />-->
-            <geometry>
-                <mesh filename="package://scout_description/meshes/scout_mini_base_link.STL" />
-            </geometry>
-        </visual>
-        <collision>
-          <!--origin
-            xyz="-0.0145261552504705 0.0231316650320557 0.00586280190939592"
-            rpy="0 0 0" /-->
-            <origin xyz="0.015 0.0231316650320557 0" rpy="0 0 0"/>
-          <geometry>
-            <mesh
-              filename="package://scout_description/meshes/scout_mini_base_link.STL" />
-          </geometry>
-        </collision>
+<robot xmlns:xacro="http://www.ros.org/wiki/xacro" name="scout_mini">
+  <!-- 参数配置 -->
+  <xacro:property name="wheel_mass" value="3"/>
+  <xacro:property name="wheel_ixx" value="0.7171"/>
+  <xacro:property name="wheel_iyy" value="0.7171"/>
+  <xacro:property name="wheel_izz" value="0.1361"/>
+  <xacro:property name="base_mass" value="30"/>
+  <xacro:property name="mesh_pkg" value="package://scout_description/meshes"/>
+  <!-- 底盘 -->
+  <link name="base_link">
+    <inertial>
+      <mass value="${base_mass}"/>
+      <origin xyz="0 0 0"/>
+      <inertia ixx="2.288641" ixy="0" ixz="0" iyy="5.103976" iyz="0" izz="3.431465"/>
+    </inertial>
+    <visual>
+      <origin rpy="1.57 0 -1.57" xyz="0 0 0.20199"/>
+      <geometry>
+        <mesh filename="${mesh_pkg}/scout_mini_base_link2.dae"/>
+      </geometry>
+    </visual>
+    <collision>
+      <origin rpy="1.57 0 -1.57" xyz="0 0 0.20199"/>
+      <geometry>
+        <mesh filename="${mesh_pkg}/scout_mini_base_link2.dae"/>
+      </geometry>
+    </collision>
+  </link>
+  <!-- 定义 wheel 宏 -->
+  <xacro:macro name="wheel" params="name parent xyz rpy axis">
+    <link name="${name}_link">
+      <inertial>
+        <mass value="${wheel_mass}"/>
+        <origin xyz="0 0 0"/>
+        <inertia ixx="${wheel_ixx}" ixy="0" ixz="0" iyy="${wheel_iyy}" iyz="0" izz="${wheel_izz}"/>
+      </inertial>
+      <visual>
+        <origin rpy="0 0 0" xyz="0 0 0"/>
+        <geometry>
+          <mesh filename="${mesh_pkg}/wheel.dae"/>
+        </geometry>
+      </visual>
+      <collision>
+        <origin rpy="0 0 0" xyz="0 0 0"/>
+        <geometry>
+          <mesh filename="${mesh_pkg}/wheel.dae"/>
+        </geometry>
+      </collision>
     </link>
-    <!-- <joint name="chassis_link_joint" type="fixed">
-        <origin xyz="0 0 ${wheel_radius - wheel_vertical_offset}" rpy="0 0 0" />
-        <parent link="base_link" />
-        <child link="chassis_link" />
-    </joint> -->
-    <link name="inertial_link">
-        <inertial>
-            <!--mass value="44.3898489950015" /-->
-            <mass value="132.3898489950015" />
-            <!-- <mass value="50" /> -->
-            <!-- <origin xyz="-0.00065 -0.085 0.062" />
-            <inertia ixx="0.6022" ixy="-0.02364" ixz="-0.1197" iyy="1.7386" iyz="-0.001544" izz="2.0296" /> -->
-            <origin xyz="0.015 0.0231316650320557 0" />
-            <!--<origin
-              xyz="-0.0145261552504705 0.0231316650320557 0.00586280190939592"
-              rpy="0 0 0" />-->
-            <inertia ixx="0.185196122711036"
-            ixy="4.30144213829512E-08"
-            ixz="5.81037523686401E-08"
-            iyy="0.364893736238929"
-            iyz="-0.000386720198091934"
-            izz="0.223868521722778" />
-            <!--<inertia ixx="2.288641" ixy="0" ixz="0" iyy="5.103976" iyz="0" izz="3.431465" />-->
-        </inertial>
-    </link>
-    <joint name="inertial_joint" type="fixed">
-        <origin xyz="0 0 0" rpy="0 0 0" />
-        <parent link="base_link" />
-        <child link="inertial_link" />
+    <joint name="${name}_joint" type="continuous">
+      <parent link="${parent}"/>
+      <child link="${name}_link"/>
+      <origin xyz="${xyz}" rpy="${rpy}"/>
+      <axis xyz="${axis}"/>
     </joint>
-    <!-- For testing, hang the robot up in the air -->
-    <!-- <link name="world" />
-    <joint name="world_to_base_link=" type="fixed">
-        <origin xyz="0 0 0.5" rpy="0 0 0" />
-        <parent link="world"/>
-        <child link="base_link"/>
-    </joint> -->
-    <!-- Scout wheel macros -->
-    <!-- wheel labeled from 0 to 3, conter-clockwise, starting from front right wheel -->
-    <!-- motor 1 and 2 (left side) are mechanically installed in a reversed direction -->
-    <xacro:scout_mini_wheel_1 wheel_prefix="front_left" wheel_diameter="${wheel_diameter}" wheel_width="${wheel_width}">
-    <!--<origin
-            xyz="0 0 0"
-            rpy="0 0 0" />-->
-        <origin xyz="${wheelbase/2} ${track/2} ${wheel_vertical_offset}" rpy="-1.57 0 0" />
-    </xacro:scout_mini_wheel_1>
-    <xacro:scout_mini_wheel_2 wheel_prefix="rear_left" wheel_diameter="${wheel_diameter}" wheel_width="${wheel_width}">
-    <!--<origin
-            xyz="0 0 0"
-            rpy="0 0 0" />-->
-        <origin xyz="${-wheelbase/2} ${track/2} ${wheel_vertical_offset}" rpy="-1.57 0 0" />
-    </xacro:scout_mini_wheel_2>
-    <xacro:scout_mini_wheel_3 wheel_prefix="front_right" wheel_diameter="${wheel_diameter}" wheel_width="${wheel_width}">
-    <!--<origin
-            xyz="0 0 0"
-            rpy="0 0 0" />-->
-        <origin xyz="${wheelbase/2} ${-track/2} ${wheel_vertical_offset+0.001}" rpy="1.57 0 0" />
-    </xacro:scout_mini_wheel_3>
-    <xacro:scout_mini_wheel_4 wheel_prefix="rear_right" wheel_diameter="${wheel_diameter}" wheel_width="${wheel_width}">
-    <!--<origin
-           xyz="0 0 0"
-           rpy="0 0 0" />-->
-        <origin xyz="${-wheelbase/2} ${-track/2} ${wheel_vertical_offset+0.001}" rpy="1.57 0 0" />
-    </xacro:scout_mini_wheel_4>
-    <!-- Additional definitions -->
-    <xacro:include filename="$(arg urdf_extras)" />
-    <!-- Gazebo definitions  -->
-    <xacro:include filename="$(find scout_description)/urdf/scout_mini.gazebo" />
+  </xacro:macro>
+  <!-- 前左轮 -->
+  <xacro:wheel name="front_left_wheel" parent="base_link"
+               xyz="0.2319755 0.2082515 0.100998" rpy="-1.57 0 0" axis="0 0 -1"/>
+  <!-- 后左轮 -->
+  <xacro:wheel name="rear_left_wheel" parent="base_link"
+               xyz="-0.2319755 0.2082515 0.100998" rpy="-1.57 0 0" axis="0 0 -1"/>
+  <!-- 前右轮 -->
+  <xacro:wheel name="front_right_wheel" parent="base_link"
+               xyz="0.2319755 -0.2082515 0.100998" rpy="1.57 0 0" axis="0 0 -1"/>
+  <!-- 后右轮 -->
+  <xacro:wheel name="rear_right_wheel" parent="base_link"
+               xyz="-0.2319755 -0.2082515 0.100998" rpy="1.57 0 0" axis="0 0 -1"/>
+  <!-- ros2_control 配置 -->
+  <ros2_control name="scout_mini_system" type="system">
+    <hardware>
+      <plugin>gz_ros2_control/GazeboSimSystem</plugin>
+    </hardware>
+    <joint name="front_left_wheel_joint">
+      <command_interface name="velocity"/>
+      <state_interface name="position"/>
+      <state_interface name="velocity"/>
+    </joint>
+    <joint name="rear_left_wheel_joint">
+      <command_interface name="velocity"/>
+      <state_interface name="position"/>
+      <state_interface name="velocity"/>
+    </joint>
+    <joint name="front_right_wheel_joint">
+      <command_interface name="velocity"/>
+      <state_interface name="position"/>
+      <state_interface name="velocity"/>
+    </joint>
+    <joint name="rear_right_wheel_joint">
+      <command_interface name="velocity"/>
+      <state_interface name="position"/>
+      <state_interface name="velocity"/>
+    </joint>
+  </ros2_control>
+  <!-- gazebo 插件 -->
+  <gazebo>
+    <plugin filename="libgz_ros2_control-system.so" name="gz_ros2_control::GazeboSimROS2ControlPlugin">
+      <parameters>$(find scout_control)/config/scout_mini_controller.yaml</parameters>
+    </plugin>
+  </gazebo>
+  <xacro:include filename="$(find scout_description)/urdf/sensor/lidar.xacro"/>
+  <xacro:lidar_sensor parent_link="base_link" xyz="0.0 0.0 0.45"/>
+  <xacro:include filename="$(find scout_description)/urdf/sensor/rgbd_camera.xacro"/>
+  <xacro:rgbd_camera_sensor parent_link="base_link" xyz= "0.24 0.0 0.32"/>
+  <xacro:include filename="$(find scout_description)/urdf/sensor/imu.xacro"/>
+  <xacro:imu_sensor parent_link="base_link" xyz= "0.0 0.0 0.15"/>
 </robot>

File: scout_description/urdf/scout_mini_backup.urdf (robot description, URDF)
Before this commit: robot scout_mini, 8 links, 7 joints
Links:
- removed link camera_link
- removed link inertial_link
- removed link laser_link
- link base_link: mass None -> 30
Joints:
- removed joint camera_joint
- removed joint inertial_joint
- removed joint laser_joint
